Commit message: modified xarm

File: xarm_description/urdf/camera2.gazebo.xacro (robot description, xacro)
@@ -1,5 +1,5 @@
 <?xml version="1.0"?>
 <robot xmlns:xacro="http://ros.org/wiki/xacro">
-  <xacro:macro name="camera_gazebo" params="prefix">
+  <xacro:macro name="camera2_gazebo" params="prefix">
     <link name="${prefix}link_camera">
       <inertial>
@@ -27,18 +27,18 @@
     </link>
     <joint
-      name="${prefix}joint_camera"
+      name="${prefix}joint_camera2"
       type="fixed">
       <origin
-        xyz="0.692 0.001 1.17"
+        xyz="0.792 0.001 1.17"
         rpy="0 1.5708 0" />
       <parent
         link="link_base" />
       <child
-        link="${prefix}link_camera" />
+        link="${prefix}link_camera2" />
     </joint>
-    <gazebo reference="${prefix}link_camera">
+    <gazebo reference="${prefix}link_camera2">
       <material>Gazebo/Black</material>
     </gazebo>
-    <gazebo reference="${prefix}link_camera">
+    <gazebo reference="${prefix}link_camera2">
       <sensor type="camera" name="xarm_camera_node">
         <update_rate>10.0</update_rate>
@@ -60,18 +60,9 @@
             <stddev>0.007</stddev>
           </noise>
-          <lens>
-          <intrinsics>
-          <fx>400</fx>
-          <fy>400</fy>
-          <cx>200</cx>
-          <cy>200</cy>
-          <s>0</s>
-          </intrinsics>
-          </lens>
         </camera>
         <plugin name="gazebo_camera" filename="libgazebo_ros_camera.so">
           <alwaysOn>true</alwaysOn>
           <updateRate>0.0</updateRate>
-          <cameraName>/camera</cameraName>
+          <cameraName>/camera2</cameraName>
           <imageTopicName>image_raw</imageTopicName>
           <cameraInfoTopicName>camera_info</cameraInfoTopicName>

File: xarm_description/urdf/xarm6.urdf.xacro (robot description, xacro)
@@ -291,4 +291,82 @@
       <dynamics damping="1.0" friction="1.0"/>
     </joint>
+    <joint name="new_camera_joint" type="fixed">
+    <axis xyz="0 1 0" />
+      <origin
+        xyz="0.692 0.201 1.17"
+        rpy="0 1.5708 0" />
+    <parent link="${prefix}link_base"/>
+    <child link="new_camera_link"/>
+  </joint>
+  <!-- Camera -->
+  <link name="new_camera_link">
+      <inertial>
+        <origin xyz="0 0 0" rpy="0 0 0" />
+        <mass value="0.1" />
+        <inertia ixx="0.01" ixy="0.0" ixz="0.0"
+                 iyy="0.01" iyz="0.0"
+                 izz="0.01" />
+      </inertial>
+      <visual>
+        <origin xyz="0 0 0" rpy="0 0 0" />
+        <geometry>
+          <sphere radius="0.02"/>
+        </geometry>
+        <material name="White">
+          <color rgba="1.0 1.0 1.0 1.0"/>
+        </material>
+      </visual>
+      <collision>
+        <origin xyz="0 0 0" rpy="0 0 0" />
+        <geometry>
+          <sphere radius="0.02"/>
+        </geometry>
+      </collision>
+  </link>
+      <gazebo reference="new_camera_link">
+    <sensor type="camera" name="camera2">
+      <update_rate>30.0</update_rate>
+      <camera name="head">
+        <horizontal_fov>0.9948376567</horizontal_fov>
+          <image>
+            <width>640</width>
+            <height>480</height>
+            <foramt>B8G8R8</foramt>
+          </image>
+          <clip>
+            <near>0.02</near>
+            <far>300</far>
+          </clip>
+          <noise>
+            <type>gaussian</type>
+            <mean>0.0</mean>
+            <stddev>0.007</stddev>
+          </noise>
+          <lens>
+          <intrinsics>
+          <fx>400</fx>
+          <fy>400</fy>
+          <cx>200</cx>
+          <cy>200</cy>
+          <s>0</s>
+          </intrinsics>
+          </lens>
+      </camera>
+      <plugin name="camera_controller" filename="libgazebo_ros_camera.so">
+        <alwaysOn>true</alwaysOn>
+        <updateRate>0.0</updateRate>
+        <cameraName>/camera2</cameraName>
+        <imageTopicName>image_raw</imageTopicName>
+        <cameraInfoTopicName>camera_info</cameraInfoTopicName>
+        <frameName>camera_link</frameName>
+        <hackBaseline>0.07</hackBaseline>
+        <distortionK1>0.0</distortionK1>
+        <distortionK2>0.0</distortionK2>
+        <distortionK3>0.0</distortionK3>
+        <distortionT1>0.0</distortionT1>
+        <distortionT2>0.0</distortionT2>
+      </plugin>
+    </sensor>
+  </gazebo>
   <xacro:if value="${rs_d435i}">
     <link name="${prefix}link_eef">

File: xarm_description/urdf/xarm6_with_gripper.xacro (robot description, xacro)
@@ -25,5 +25,8 @@
     </xacro:kinect_v2> -->
     <xacro:include filename="$(find xarm_description)/urdf/camera.gazebo.xacro" />
+    <xacro:include filename="$(find xarm_description)/urdf/camera2.gazebo.xacro" />
     <xacro:camera_gazebo prefix="$(arg prefix)" />
+      <!--<xacro:camera_gazebo prefix="camera1" /> -->
+    <!-- <xacro:camera2_gazebo prefix="camera2" /> -->
   </xacro:if>
 </robot>

File: xarm_gripper/urdf/xarm_gripper.gazebo.xacro (robot description, xacro)
@@ -5,7 +5,7 @@
     <gazebo>
       <!-- old version -->
-      <plugin name="${name_prefix}mimic_joint_plugin" filename="libroboticsgroup_gazebo_mimic_joint_plugin.so">
+          <!--   <plugin name="${name_prefix}mimic_joint_plugin" filename="libroboticsgroup_gazebo_mimic_joint_plugin.so"> -->
       <!-- new version -->
-      <!-- <plugin name="${name_prefix}mimic_joint_plugin" filename="libroboticsgroup_upatras_gazebo_mimic_joint_plugin.so"> -->
+      <plugin name="${name_prefix}mimic_joint_plugin" filename="libroboticsgroup_upatras_gazebo_mimic_joint_plugin.so">
         <joint>${following_joint}</joint>
         <mimicJoint>${mimic_joint}</mimicJoint>
